File: rusEFI-Optoisolator/rusEFI-Optoisolator.kicad_sch (KiCad schematic)
At the start: 11 parts, among them J1 Conn_01x02_Male, J2 Conn_01x03_Male, U1 4N25

Commit message: Updates, gerbers and bom files.
Parts:
- C1: LCSC (none) -> C469523
- C2: footprint Capacitor_SMD:C_0805_2012Metric -> Capacitor_SMD:C_1206_3216Metric; LCSC (none) -> C77494
- D2: LCSC (none) -> C134432
- D4: LCSC (none) -> C2903856
- R1: footprint Resistor_SMD:R_0805_2012Metric -> Resistor_SMD:R_1206_3216Metric; LCSC (none) -> C2759146
- R2: LCSC (none) -> C2907326
- U1: LCSC (none) -> C3008818
Changed lines of the file:
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@@
+      (effects (font (size 1.27 1.27)) hide)
+    )
+    (property "LCSC" "C2907326" (id 4) (at 152.4 63.5 90)
       (effects (font (size 1.27 1.27)) hide)
     )
@@
     )
     (property "Datasheet" "~" (id 3) (at 92.71 63.5 0)
+      (effects (font (size 1.27 1.27)) hide)
+    )
+    (property "LCSC" "C2903856" (id 4) (at 92.71 63.5 0)
       (effects (font (size 1.27 1.27)) hide)
     )
@@
       (effects (font (size 1.27 1.27)) (justify left) hide)
     )
+    (property "LCSC" "C3008818" (id 4) (at 121.92 66.04 0)
+      (effects (font (size 1.27 1.27)) hide)
+    )
     (pin "1")
     (pin "2")
@@
       (effects (font (size 1.27 1.27)) hide)
     )
+    (property "LCSC" "C134432" (id 4) (at 72.39 63.5 0)
+      (effects (font (size 1.27 1.27)) hide)
+    )
     (pin "1")
     (pin "2")
@@
     (property "Reference" "R1" (id 0) (at 82.55 57.15 90))
     (property "Value" "390" (id 1) (at 82.55 59.69 90))
-    (property "Footprint" "Resistor_SMD:R_0805_2012Metric" (id 2) (at 82.55 65.278 90)
+    (property "Footprint" "Resistor_SMD:R_1206_3216Metric" (id 2) (at 82.55 65.278 90)
       (effects (font (size 1.27 1.27)) hide)
     )
     (property "Datasheet" "~" (id 3) (at 82.55 63.5 0)
+      (effects (font (size 1.27 1.27)) hide)
+    )
+    (property "LCSC" "C2759146" (id 4) (at 82.55 63.5 90)
       (effects (font (size 1.27 1.27)) hide)
     )
@@
       (effects (font (size 1.27 1.27)) hide)
     )
+    (property "LCSC" "C469523" (id 4) (at 142.24 68.58 90)
+      (effects (font (size 1.27 1.27)) hide)
+    )
     (pin "1")
     (pin "2")
@@
       (effects (font (size 1.27 1.27)) (justify left))
     )
-    (property "Footprint" "Capacitor_SMD:C_0805_2012Metric" (id 2) (at 101.6 68.58 0)
+    (property "Footprint" "Capacitor_SMD:C_1206_3216Metric" (id 2) (at 101.6 68.58 0)
       (effects (font (size 1.27 1.27)) hide)
     )
     (property "Datasheet" "~" (id 3) (at 101.6 68.58 0)
+      (effects (font (size 1.27 1.27)) hide)
+    )
+    (property "LCSC" "C77494" (id 4) (at 101.6 68.58 0)
       (effects (font (size 1.27 1.27)) hide)
     )
@@
     )
     (path "/b04ef9c6-d45d-4dee-b840-f4030944323a"
-      (reference "C2") (unit 1) (value "0.001uF1") (footprint "Capacitor_SMD:C_0805_2012Metric")
+      (reference "C2") (unit 1) (value "0.001uF1") (footprint "Capacitor_SMD:C_1206_3216Metric")
     )
     (path "/cae3c730-c1b3-4b1f-b4f5-2e236a32eefe"
@@
     )
     (path "/8ff3f878-da75-4ba0-8a5c-92128a3f6039"
-      (reference "R1") (unit 1) (value "390") (footprint "Resistor_SMD:R_0805_2012Metric")
+      (reference "R1") (unit 1) (value "390") (footprint "Resistor_SMD:R_1206_3216Metric")
     )
     (path "/4c387d21-8555-4529-bedb-aff458b46c9a"

Commit message: New version
Parts:
- removed D3: DNP, Diode_SMD:D_SMA, symbol Device:D_Zener
- removed D4: 1SMA4748A, Diode_SMD:D_SMA, symbol Device:D_Zener
- added C3: 0.22uF, Capacitor_SMD:C_1206_3216Metric, symbol Device:C_Small
- C2: value 0.001uF1 -> 0.001uF
- D1: value DNP -> 1SMA4748A; LCSC (none) -> C2903856
- R1: footprint Resistor_SMD:R_1206_3216Metric -> Resistor_THT:R_Axial_DIN0207_L6.3mm_D2.5mm_P15.24mm_Horizontal
Connections:
- net Coil_in: no longer D1.1 (K)
- net GND: now also C3.2; no longer D1.2 (A)
- net Trigger_Output: now also U1.5; no longer U1.6
- net at R1.2: now also C2.1, U1.1
- net at R1.1: now also D1.2 (A), C3.1; no longer D2.1 (K)
- new net: D1.1 (K), D2.1 (K)

Commit message: update
Connections:
- net GND: no longer C2.2, C3.2, J1.2 (Pin_2), U1.2
- new net: C2.2, C3.2, J1.2 (Pin_2), U1.2
Changed lines of the file:
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@@
-    (stroke (width 0) (type default) (color 0 0 0 0))
-  )
-  (wire (pts (xy 66.04 71.12) (xy 66.04 72.39))
     (stroke (width 0) (type default) (color 0 0 0 0))
   )
@@
     (stroke (width 0) (type default) (color 0 0 0 0))
   )
-  (wire (pts (xy 66.04 72.39) (xy 66.097 72.39))
-    (stroke (width 0) (type default) (color 0 0 0 0))
-  )
